File: esp32_engine_starter/hardware/hijet_starter.kicad_pcb (KiCad board)
At the start: 2 copper layers, 98 x 90 mm, 57 parts, among them J1 12V IN, J2 OUT, J3 IN, J4 I2C, J5 ESP32 VIN row, J6 ESP32 3V3 row, J7 OBD-II CAN, J8 GPS, Q1 2SC1815, U1 M78AR05-1, U2 PC817, U3 PC817, U4 PC817, U5 PC817, U6 PC817, U7 PC817, U8 PC817, U9 MCP2562-E/P

Commit message: 電圧測定の R2 を 18k から 10k に変更（組み立て時の手持ちに合わせる）
config.h の分圧比を (100+10)/10 に変更。16V で 1.46V、9V で 0.82V と
ADC の精度範囲内。シミュレーションに下限 0.15V の確認を追加。全検証合格。

Co-Authored-By: Claude Opus 5.5 <noreply@anthropic.com>
Claude-Session: https://claude.ai/code/session_011cXkDUypHbxixpJEznYmeT
Parts:
- R2: value 18k -> 10k
